File: ADC_12_channel.sch (EAGLE design)
At the start: 166 parts, among them IC1 LM317BD2T, IC2 LM317BD2T, K1 691131710003, K2 691101710002, K3 691101710002, K4 691101710002, K5 691101710002, K6 691101710002, K7 691101710002, K8 691101710002, K9 691101710002, Q1 L78M12ABDT, U1 AD7864ASZ-1, U10 TL082D, U12 V_REG_317SMD, U2 AD7864ASZ-1, U3 TL082D, U4 TL082D, U5 TL082D, U6 TL082D, U7 TL082D, U8 TL082D, U9 TL082D, X1 QTE-040

Commit message: Finished Ground plane and supply
Connections:
- net VDD: now also U1.~STBY, U2.~STBY
Other:
- moved on the sheet: CLK_IN, CONVST1, R20
Changed lines of the file:
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@@
 <instance part="R10" gate="G$1" x="-43.18" y="-124.46" rot="R180"/>
 <instance part="DVDD3" gate="G$1" x="-53.34" y="-124.46" rot="R90"/>
-<instance part="CLK_IN" gate="1" x="-5.08" y="55.88"/>
+<instance part="CLK_IN" gate="1" x="-2.54" y="55.88"/>
 <instance part="U3" gate="A" x="-274.32" y="119.38"/>
 <instance part="U3" gate="B" x="-223.52" y="121.92"/>
@@
 <instance part="AGND2" gate="GND" x="17.78" y="27.94" rot="R270"/>
 <instance part="GND6" gate="1" x="5.08" y="53.34" rot="R270"/>
-<instance part="SUPPLY3" gate="GND" x="10.16" y="58.42" rot="R270"/>
+<instance part="SUPPLY3" gate="GND" x="7.62" y="58.42" rot="R270"/>
 <instance part="D1" gate="G$1" x="589.28" y="274.32"/>
 <instance part="D2" gate="G$1" x="589.28" y="243.84"/>
@@
 <instance part="R70" gate="G$1" x="236.22" y="-12.7" rot="R90"/>
 <instance part="U12" gate="G$1" x="754.38" y="274.32"/>
-<instance part="CONVST1" gate="1" x="0" y="58.42" rot="R90"/>
-<instance part="R20" gate="G$1" x="-7.62" y="60.96" rot="R180"/>
+<instance part="CONVST1" gate="1" x="-7.62" y="58.42" rot="R90"/>
+<instance part="R20" gate="G$1" x="-17.78" y="60.96" rot="R180"/>
 <instance part="R72" gate="G$1" x="-38.1" y="-111.76" rot="R180"/>
 <instance part="IC1" gate="G$1" x="617.22" y="243.84" rot="R180"/>
@@
 <net name="N$1" class="0">
 <segment>
-<pinref part="U1" gate="A" pin="DB0"/>
-<wire x1="76.2" y1="83.82" x2="81.28" y2="83.82" width="0.1524" layer="91"/>
 <pinref part="X1" gate="-12" pin="1"/>
 <pinref part="U2" gate="A" pin="DB0"/>
@@
 <wire x1="76.2" y1="-91.44" x2="81.28" y2="-91.44" width="0.1524" layer="91"/>
 <wire x1="81.28" y1="-91.44" x2="81.28" y2="83.82" width="0.1524" layer="91"/>
+<pinref part="U1" gate="A" pin="DB0"/>
+<wire x1="76.2" y1="83.82" x2="81.28" y2="83.82" width="0.1524" layer="91"/>
 <junction x="81.28" y="83.82"/>
 </segment>
@@
 <pinref part="C5" gate="G$1" pin="2"/>
 </segment>
+<segment>
+<pinref part="U1" gate="A" pin="~STBY"/>
+<label x="10.16" y="68.58" size="1.778" layer="95" rot="R180" xref="yes"/>
+<wire x1="25.4" y1="68.58" x2="10.16" y2="68.58" width="0.1524" layer="91"/>
+</segment>
+<segment>
+<pinref part="U2" gate="A" pin="~STBY"/>
+<wire x1="25.4" y1="-106.68" x2="10.16" y2="-106.68" width="0.1524" layer="91"/>
+<label x="10.16" y="-106.68" size="1.778" layer="95" rot="R180" xref="yes"/>
+</segment>
 </net>
 <net name="N$16" class="0">
@@
 <pinref part="CLK_IN" gate="1" pin="P"/>
 <pinref part="U1" gate="A" pin="CLKIN"/>
-<wire x1="-2.54" y1="55.88" x2="25.4" y2="55.88" width="0.1524" layer="91"/>
+<wire x1="0" y1="55.88" x2="25.4" y2="55.88" width="0.1524" layer="91"/>
 </segment>
 </net>
@@
 </segment>
 <segment>
-<wire x1="-215.9" y1="121.92" x2="-218.44" y2="121.92" width="0.1524" layer="91"/>
 <wire x1="-215.9" y1="121.92" x2="-210.82" y2="121.92" width="0.1524" layer="91"/>
 <pinref part="U3" gate="B" pin="OUT"/>
-<junction x="-215.9" y="121.92"/>
 <pinref part="R37" gate="G$1" pin="1"/>
 <wire x1="-210.82" y1="121.92" x2="-203.2" y2="121.92" width="0.1524" layer="91"/>
@@
 <wire x1="-215.9" y1="104.14" x2="-215.9" y2="109.22" width="0.1524" layer="91"/>
 <junction x="-215.9" y="109.22"/>
+<label x="-205.74" y="121.92" size="1.778" layer="95" rot="R270" xref="yes"/>
 </segment>
 </net>
@@
 <segment>
 <pinref part="R20" gate="G$1" pin="2"/>
-<wire x1="-12.7" y1="60.96" x2="-15.24" y2="60.96" width="0.1524" layer="91"/>
-<label x="-15.24" y="60.96" size="1.778" layer="95" rot="R270" xref="yes"/>
+<wire x1="-22.86" y1="60.96" x2="-22.86" y2="58.42" width="0.1524" layer="91"/>
+<label x="-22.86" y="58.42" size="1.778" layer="95" rot="R270" xref="yes"/>
 </segment>
 <segment>
@@
 <wire x1="-22.86" y1="-114.3" x2="-22.86" y2="-119.38" width="0.1524" layer="91"/>
 <label x="-22.86" y="-119.38" size="1.778" layer="95" rot="R270" xref="yes"/>
-</segment>
-</net>
-<net name="N$49" class="0">
-<segment>
-<wire x1="309.88" y1="-53.34" x2="309.88" y2="-50.8" width="0.1524" layer="91"/>
 </segment>
 </net>
@@
 <pinref part="X1" gate="-28" pin="1"/>
 <wire x1="251.46" y1="63.5" x2="302.26" y2="63.5" width="0.1524" layer="91"/>
-</segment>
-</net>
-<net name="N$51" class="0">
-<segment>
-<wire x1="132.08" y1="-27.94" x2="129.54" y2="-27.94" width="0.1524" layer="91"/>
-<wire x1="129.54" y1="-27.94" x2="129.54" y2="-25.4" width="0.1524" layer="91"/>
 </segment>
 </net>
@@
 <wire x1="680.72" y1="266.7" x2="680.72" y2="256.54" width="0.1524" layer="91"/>
 <junction x="680.72" y="256.54"/>
+<label x="716.28" y="254" size="1.778" layer="95" rot="R270" xref="yes"/>
 </segment>
 <segment>
@@
 <segment>
 <pinref part="C2" gate="G$1" pin="1"/>
-<wire x1="15.24" y1="58.42" x2="12.7" y2="58.42" width="0.1524" layer="91"/>
+<wire x1="15.24" y1="58.42" x2="10.16" y2="58.42" width="0.1524" layer="91"/>
 <pinref part="SUPPLY3" gate="GND" pin="GND"/>
 </segment>
@@
 <pinref part="R20" gate="G$1" pin="1"/>
 <pinref part="CONVST1" gate="1" pin="P"/>
-<wire x1="-2.54" y1="60.96" x2="0" y2="60.96" width="0.1524" layer="91"/>
+<wire x1="-12.7" y1="60.96" x2="-7.62" y2="60.96" width="0.1524" layer="91"/>
 <pinref part="U1" gate="A" pin="~CONVST"/>
-<wire x1="0" y1="60.96" x2="25.4" y2="60.96" width="0.1524" layer="91"/>
-<junction x="0" y="60.96"/>
+<wire x1="-7.62" y1="60.96" x2="25.4" y2="60.96" width="0.1524" layer="91"/>
+<junction x="-7.62" y="60.96"/>
 </segment>
 </net>
@@
 </sheet>
 </sheets>
+<errors>
+</errors>
 </schematic>
 </drawing>
